File: modern-keyboard-template/modern-keyboard-template.kicad_sch (KiCad schematic)
At the start: 26 parts, among them J1 USB_C_Receptacle_USB2.0, J2 Conn_01x05, J3 Conn_01x04, U1 STM32F072CBT6, U2 PRTR5V0U2X, U3 XC6206PxxxMR-Regulator_Linear, U5 TXB0101

Commit message: created matrix sheet
Parts:
- removed J3: Conn_01x04, KiCad-SSD1306-0.91-OLED-4pin-128x32.pretty-master:SSD1306-0.91-OLED-4pin-128x32, symbol Connector_Generic:Conn_01x04
Other:
- added sheet matrix (matrix.kicad_sch)
- note removed: "OLED Display Intended to be used with the SSD1306 128x32 pixel display."
